File: Hardware/SparkFun_LSM303C_6_DOF_IMU_Breakout.sch (EAGLE design)
At the start: 23 parts, among them Q1 2.5A/30V, U1 LSM303C, U2 10ms

Commit message: Ready for proto review
Parts:
- JP1: device SparkFun-Connectors:M06SILK_FEMALE_PTH -> SparkFun-Connectors:I2C_STANDARD
- JP2: device SparkFun-Connectors:M04PTH -> SparkFun-Connectors:M06SILK_FEMALE_PTH
- SJ1: value JUMPER-PAD-2-NO -> JUMPER-PAD-3-NOYES_SILK; device SparkFun-Passives:JUMPER-PAD-2-NO -> SparkFun-Passives:JUMPER-PAD-3-NOYES_SILK
- U2: value 10ms -> LM3880
Connections:
- new net N$2: R2.2, SJ1.3
- new net SCL/SCLK: JP1.4, U1.SCL/SPC
- new net SDA/SDI/SDO: JP1.3, U1.SDA/SDI/SDO
- net CLOCK: no longer JP2.4, U1.SCL/SPC
- net CS_MAG: now also JP2.5; no longer JP2.2
- net DRDY_MAG: now also JP2.2; no longer JP1.2
- net GND: now also JP1.1, R3.2; no longer JP1.5, SJ2.1
- net I2C-UP: no longer R2.2
- net INT_MAG: now also JP2.6; no longer JP1.6
- net INT_XL: now also JP2.1; no longer JP1.1
- net N$3: now also U2.!F1; no longer U2.!2
- net SD: no longer JP2.1, U1.SDA/SDI/SDO
- net VCC: now also JP2.4; no longer JP1.4
- net VDD_IO: now also JP1.2, SJ2.1; no longer JP1.3, R3.2
Other:
- note added: "2 ms DELAY ON VDD"
- note added: "Each output adds a 2ms delay (AE). Using flag 1 to delay VDD 2ms from VDD_IO."
- note removed: "20 ms DELAY ON VDD"
- moved on the sheet: Q1, R1, R3, SJ2, U2
